File: hardware/DaisySeedThingie.kicad_sch (KiCad schematic)
At the start: 66 parts, among them J1 LEDS, J10 AUDIO IN LR, J11 AUDIO IN L, J12 AUDIO IN R, J13 AUDIO OUT LR, J14 AUDIO OUT L, J15 AUDIO OUT R, J16 MIDI IN, J17 MIDI OUT, J18 MIDI IN, J19 MIDI OUT, J2 DC IN, J20 A, J21 B, J22 C, J23 D, J3 DAISY PINS, J4 COMPONENTS, J5 DAISY PINS, J6 Yamaichi PJS008-4100-0-VE, J7 MICRO SD, J8 AUDIO IN, J9 AUDIO OUT, SW1 ENCODER, SW2 A, SW3 C, SW4 B, SW5 D, U1 DAISY SEED, U2 H11L1, U3 128x64

Commit message: Restore after bad merge
Parts:
- D1: value A -> RED; Label (none) -> A
- D2: value B -> RED; Label (none) -> B
- F1: value Fuse -> 5x20mm; Label (none) -> Fuse
- J1: value LEDS -> 01x02 PIN CONNECTOR; Label (none) -> LEDS
- J10: value AUDIO IN LR -> STEREO 3.5mm; Display 3.5mm_Stereo -> (none); Label (none) -> IN LR
- J11: value AUDIO IN L -> MONO 3.5mm; Display 3.5mm_Mono -> (none); Label (none) -> IN L
- J12: value AUDIO IN R -> MONO 3.5mm; Display 3.5mm_Mono -> (none); Label (none) -> IN R
- J13: value AUDIO OUT LR -> STEREO 3.5mm; Display 3.5mm_Stereo -> (none); Label (none) -> OUT LR
- J14: value AUDIO OUT L -> MONO 3.5mm; Display 3.5mm_Mono -> (none); Label (none) -> OUT L
- J15: value AUDIO OUT R -> MONO 3.5mm; Display 3.5mm_Mono -> (none); Label (none) -> OUT R
- J16: value MIDI IN -> STEREO 3.5mm; Display 3.5mm_Stereo -> (none); Label (none) -> MIDI IN
- J17: value MIDI OUT -> STEREO 3.5mm; Display 3.5mm_Stereo -> (none); Label (none) -> MIDI OUT
- J18: value MIDI IN -> JST 01x03; Label (none) -> MIDI IN
- J19: value MIDI OUT -> JST 01x03; Label (none) -> MIDI OUT
- J2: value DC IN -> DC Barrel Jack
- J20: value A -> MONO 3.5mm; Display A -> (none); Label (none) -> A
- J21: value B -> MONO 3.5mm; Display B -> (none); Label (none) -> B
- J22: value C -> MONO 3.5mm; Display C -> (none); Label (none) -> C
- J23: value D -> MONO 3.5mm; Display D -> (none); Label (none) -> D
- J3, J5: value DAISY PINS -> 02x20 PIN CONNECTOR; Label (none) -> DAISY PINS
- J4: value COMPONENTS -> 02x17 PIN CONNECTOR; Label (none) -> COMPONENTS
- J7: value MICRO SD -> 01x06 PIN CONNECTOR; Label (none) -> MICRO SD
- J8: value AUDIO IN -> JST 01x03; Label (none) -> AUDIO IN
- J9: value AUDIO OUT -> JST 01x03; Label (none) -> AUDIO OUT
- JP1, JP4: value MIDI_B -> JUMPER; Label (none) -> MIDI B
- JP2, JP3: value MIDI_A -> JUMPER; Label (none) -> MIDI A
- RV1: footprint Desval:Potentiometer_Alpha_RD901F-40-00D_Single_Vertical -> Desval:Potentiometer_Alps_RK09K_Single_Vertical; symbol Device:R_Potentiometer -> Device:R_Potentiometer_MountingPin; Display A -> (none); Label (none) -> A
- RV2: footprint Desval:Potentiometer_Alpha_RD901F-40-00D_Single_Vertical -> Desval:Potentiometer_Alps_RK09K_Single_Vertical; symbol Device:R_Potentiometer -> Device:R_Potentiometer_MountingPin; Display B -> (none); Label (none) -> B
- RV3: footprint Desval:Potentiometer_Alpha_RD901F-40-00D_Single_Vertical -> Desval:Potentiometer_Alps_RK09K_Single_Vertical; symbol Device:R_Potentiometer -> Device:R_Potentiometer_MountingPin; Display C -> (none); Label (none) -> C
- RV4: footprint Desval:Potentiometer_Alpha_RD901F-40-00D_Single_Vertical -> Desval:Potentiometer_Alps_RK09K_Single_Vertical; symbol Device:R_Potentiometer -> Device:R_Potentiometer_MountingPin; Display D -> (none); Label (none) -> D
- S1: value POWER -> EG2219; Label (none) -> POWER
- SW1: value ENCODER -> EN11C; Label (none) -> ENCODER
- SW2: value A -> SW_PUSH_6mm; Label (none) -> A
- SW3: value C -> SW_PUSH_6mm; Label (none) -> C
- SW4: value B -> SW_PUSH_6mm; Label (none) -> B
- SW5: value D -> SW_PUSH_6mm; Label (none) -> D
- U3: value 128x64 -> SSD1306 0.96" OLED I2C; Label (none) -> DISPLAY
Connections:
- net GND: now also RV1.MP (MountPin), RV2.MP (MountPin), RV3.MP (MountPin), RV4.MP (MountPin), S1.S1 (SHIELD), S1.S2 (SHIELD), S1.S3 (SHIELD), S1.S4 (SHIELD)
- new net: J2.2, S1.5
Other:
- moved on the sheet: D1, D2, F1, J1, R1, R2

Commit message: Initial Revision B
Parts:
- removed H5: MountingHole_Pad, MountingHole:MountingHole_3.2mm_M3_Pad, symbol Mechanical:MountingHole_Pad
Changed lines of the file:
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@@
 	(title_block
 		(title "Daisy Seed Thingie")
+		(date "2026-04-06")
+		(rev "B")
 		(company "The House of Galahad")
 	)
@@
 	(symbol
 		(lib_id "power:GND")
-		(at 40.64 55.88 0)
-		(unit 1)
-		(exclude_from_sim no)
-		(in_bom yes)
-		(on_board yes)
-		(dnp no)
-		(fields_autoplaced yes)
-		(property "Reference" "#PWR065"
-			(at 40.64 62.23 0)
-			(effects
-				(font
-					(size 1.27 1.27)
-				)
-				(hide yes)
-			)
-		)
-		(property "Value" "GND"
-			(at 40.64 60.96 0)
-			(effects
-				(font
-					(size 1.27 1.27)
-				)
-			)
-		)
-		(property "Footprint" ""
-			(at 40.64 55.88 0)
-			(effects
-				(font
-					(size 1.27 1.27)
-				)
-				(hide yes)
-			)
-		)
-		(property "Datasheet" ""
-			(at 40.64 55.88 0)
-			(effects
-				(font
-					(size 1.27 1.27)
-				)
-				(hide yes)
-			)
-		)
-		(property "Description" "Power symbol creates a global label with name \"GND\" , ground"
-			(at 40.64 55.88 0)
-			(effects
-				(font
-					(size 1.27 1.27)
-				)
-				(hide yes)
-			)
-		)
-		(pin "1"
-		)
-		(instances
-			(project "DaisySeedThingie"
-				(path "/e16aa8e8-029e-4c85-96a5-88f157e594bc"
-					(reference "#PWR065")
-					(unit 1)
-				)
-			)
-		)
-	)
-	(symbol
-		(lib_id "power:GND")
 		(at 97.79 148.59 0)
 		(unit 1)
@@
 					(unit 1)
 				)
-			)
-		)
-	)
-	(symbol
-		(lib_id "Mechanical:MountingHole_Pad")
-		(at 40.64 53.34 0)
-		(unit 1)
-		(exclude_from_sim no)
-		(in_bom no)
-		(on_board yes)
-		(dnp no)
-		(fields_autoplaced yes)
-		(property "Reference" "H5"
-			(at 43.18 50.7999 0)
-			(effects
-				(font
-					(size 1.27 1.27)
-				)
-				(justify left)
-			)
-		)
-		(property "Value" "MountingHole_Pad"
-			(at 43.18 53.3399 0)
-			(effects
-				(font
-					(size 1.27 1.27)
-				)
-				(justify left)
-			)
-		)
-		(property "Footprint" "MountingHole:MountingHole_3.2mm_M3_Pad"
-			(at 40.64 53.34 0)
-			(effects
-				(font
-					(size 1.27 1.27)
-				)
-				(hide yes)
-			)
-		)
-		(property "Datasheet" "~"
-			(at 40.64 53.34 0)
-			(effects
-				(font
-					(size 1.27 1.27)
-				)
-				(hide yes)
-			)
-		)
-		(property "Description" "Mounting Hole with connection"
-			(at 40.64 53.34 0)
-			(effects
-				(font
-					(size 1.27 1.27)
-				)
-				(hide yes)
-			)
-		)
-		(pin "1"
-		)
-		(instances
-			(project "DaisySeedThingie"
-				(path "/e16aa8e8-029e-4c85-96a5-88f157e594bc"
-					(reference "H5")
-					(unit 1)
-				)
